File: AtTinyRaw_1/AtTinyRaw_1.kicad_sch (KiCad schematic)
At the start: 12 parts, among them J1 Power, J2 PinOut, J3 USB_B_Micro, U1 ATtiny85-20S, U2 L7805

Commit message: Update
Parts:
- added J4: Power, Connector_PinSocket_2.54mm:PinSocket_1x03_P2.54mm_Vertical, symbol Connector:Conn_01x03_Male
- added J5: PinOut, Connector_PinSocket_2.54mm:PinSocket_1x06_P2.54mm_Vertical, symbol Connector:Conn_01x06_Male
Connections:
- net +5V: now also J4.3 (Pin_3)
- net +VDC: now also J4.1 (Pin_1)
- net GND: now also J4.2 (Pin_2)
- net PB0: now also J5.6 (Pin_6)
- net PB1: now also J5.5 (Pin_5)
- net PB2: now also J5.4 (Pin_4)
- net PB3: now also J5.3 (Pin_3)
- net PB4: now also J5.2 (Pin_2)
- net PB5: now also J5.1 (Pin_1)
Other:
- moved on the sheet: J1
Changed lines of the file:
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@@
   (junction (at 135.89 153.67) (diameter 0) (color 0 0 0 0)
   )
+  (junction (at 175.895 111.76) (diameter 0) (color 0 0 0 0)
+  )
   (junction (at 186.69 144.78) (diameter 0) (color 0 0 0 0)
   )
+  (junction (at 175.895 114.3) (diameter 0) (color 0 0 0 0)
+  )
   (junction (at 161.29 111.76) (diameter 0) (color 0 0 0 0)
   )
@@
   (junction (at 139.7 153.67) (diameter 0) (color 0 0 0 0)
   )
+  (junction (at 147.32 137.795) (diameter 0) (color 0 0 0 0)
+  )
   (junction (at 149.86 166.37) (diameter 0) (color 0 0 0 0)
   )
   (junction (at 186.69 127) (diameter 0) (color 0 0 0 0)
   )
+  (junction (at 175.895 101.6) (diameter 0) (color 0 0 0 0)
+  )
   (junction (at 163.83 109.22) (diameter 0) (color 0 0 0 0)
   )
+  (junction (at 149.86 137.795) (diameter 0) (color 0 0 0 0)
+  )
+  (junction (at 175.895 109.22) (diameter 0) (color 0 0 0 0)
+  )
+  (junction (at 175.895 106.68) (diameter 0) (color 0 0 0 0)
+  )
+  (junction (at 175.895 104.14) (diameter 0) (color 0 0 0 0)
+  )
   (junction (at 184.15 129.54) (diameter 0) (color 0 0 0 0)
   )
+  (junction (at 152.4 137.795) (diameter 0) (color 0 0 0 0)
+  )
   (junction (at 161.29 153.67) (diameter 0) (color 0 0 0 0)
   )
@@
     (stroke (width 0) (type default) (color 0 0 0 0))
   )
-  (wire (pts (xy 153.67 106.68) (xy 189.23 106.68))
+  (wire (pts (xy 153.67 106.68) (xy 175.895 106.68))
+    (stroke (width 0) (type default) (color 0 0 0 0))
+  )
+  (wire (pts (xy 152.4 137.795) (xy 152.4 142.24))
     (stroke (width 0) (type default) (color 0 0 0 0))
   )
@@
     (stroke (width 0) (type default) (color 0 0 0 0))
   )
+  (wire (pts (xy 175.895 111.76) (xy 189.23 111.76))
+    (stroke (width 0) (type default) (color 0 0 0 0))
+  )
   (wire (pts (xy 184.15 124.46) (xy 184.15 129.54))
     (stroke (width 0) (type default) (color 0 0 0 0))
@@
     (stroke (width 0) (type default) (color 0 0 0 0))
   )
+  (wire (pts (xy 175.895 114.3) (xy 189.23 114.3))
+    (stroke (width 0) (type default) (color 0 0 0 0))
+  )
   (wire (pts (xy 161.29 153.67) (xy 161.29 156.21))
     (stroke (width 0) (type default) (color 0 0 0 0))
@@
     (stroke (width 0) (type default) (color 0 0 0 0))
   )
+  (wire (pts (xy 175.895 106.68) (xy 189.23 106.68))
+    (stroke (width 0) (type default) (color 0 0 0 0))
+  )
   (wire (pts (xy 152.4 142.24) (xy 158.75 142.24))
     (stroke (width 0) (type default) (color 0 0 0 0))
@@
     (stroke (width 0) (type default) (color 0 0 0 0))
   )
-  (wire (pts (xy 161.29 111.76) (xy 189.23 111.76))
+  (wire (pts (xy 161.29 111.76) (xy 175.895 111.76))
     (stroke (width 0) (type default) (color 0 0 0 0))
   )
@@
     (stroke (width 0) (type default) (color 0 0 0 0))
   )
-  (wire (pts (xy 153.67 104.14) (xy 189.23 104.14))
+  (wire (pts (xy 153.67 104.14) (xy 175.895 104.14))
     (stroke (width 0) (type default) (color 0 0 0 0))
   )
@@
     (stroke (width 0) (type default) (color 0 0 0 0))
   )
+  (wire (pts (xy 149.86 137.795) (xy 149.86 138.43))
+    (stroke (width 0) (type default) (color 0 0 0 0))
+  )
   (wire (pts (xy 199.39 137.16) (xy 199.39 144.78))
     (stroke (width 0) (type default) (color 0 0 0 0))
   )
+  (wire (pts (xy 147.32 137.795) (xy 147.32 144.78))
+    (stroke (width 0) (type default) (color 0 0 0 0))
+  )
   (wire (pts (xy 170.18 129.54) (xy 161.29 129.54))
     (stroke (width 0) (type default) (color 0 0 0 0))
@@
     (stroke (width 0) (type default) (color 0 0 0 0))
   )
-  (wire (pts (xy 163.83 109.22) (xy 189.23 109.22))
+  (wire (pts (xy 163.83 109.22) (xy 175.895 109.22))
     (stroke (width 0) (type default) (color 0 0 0 0))
   )
@@
     (stroke (width 0) (type default) (color 0 0 0 0))
   )
-  (wire (pts (xy 153.67 114.3) (xy 189.23 114.3))
+  (wire (pts (xy 153.67 114.3) (xy 175.895 114.3))
     (stroke (width 0) (type default) (color 0 0 0 0))
   )
@@
     (stroke (width 0) (type default) (color 0 0 0 0))
   )
+  (wire (pts (xy 175.895 109.22) (xy 189.23 109.22))
+    (stroke (width 0) (type default) (color 0 0 0 0))
+  )
+  (wire (pts (xy 175.895 101.6) (xy 189.23 101.6))
+    (stroke (width 0) (type default) (color 0 0 0 0))
+  )
   (wire (pts (xy 161.29 161.29) (xy 161.29 166.37))
     (stroke (width 0) (type default) (color 0 0 0 0))
@@
     (stroke (width 0) (type default) (color 0 0 0 0))
   )
-  (wire (pts (xy 147.32 137.16) (xy 147.32 144.78))
+  (wire (pts (xy 147.32 133.35) (xy 147.32 137.795))
     (stroke (width 0) (type default) (color 0 0 0 0))
   )
@@
     (stroke (width 0) (type default) (color 0 0 0 0))
   )
-  (wire (pts (xy 153.67 101.6) (xy 189.23 101.6))
+  (wire (pts (xy 153.67 101.6) (xy 175.895 101.6))
     (stroke (width 0) (type default) (color 0 0 0 0))
   )
@@
     (stroke (width 0) (type default) (color 0 0 0 0))
   )
-  (wire (pts (xy 149.86 137.16) (xy 149.86 138.43))
+  (wire (pts (xy 149.86 133.35) (xy 149.86 137.795))
     (stroke (width 0) (type default) (color 0 0 0 0))
   )
@@
     (stroke (width 0) (type default) (color 0 0 0 0))
   )
+  (wire (pts (xy 175.895 104.14) (xy 189.23 104.14))
+    (stroke (width 0) (type default) (color 0 0 0 0))
+  )
   (wire (pts (xy 175.26 129.54) (xy 184.15 129.54))
     (stroke (width 0) (type default) (color 0 0 0 0))
   )
-  (wire (pts (xy 152.4 137.16) (xy 152.4 142.24))
+  (wire (pts (xy 152.4 133.35) (xy 152.4 137.795))
     (stroke (width 0) (type default) (color 0 0 0 0))
   )
@@
   (label "PB4" (at 166.37 111.76 0)
     (effects (font (size 1.27 1.27)) (justify left bottom))
+  )
+  (symbol (lib_id "Connector:Conn_01x06_Male") (at 180.975 109.22 180) (unit 1)
+    (in_bom yes) (on_board yes) (fields_autoplaced)
+    (property "Reference" "J5" (id 0) (at 182.245 109.2201 0)
+      (effects (font (size 1.27 1.27)) (justify right))
+    )
+    (property "Value" "PinOut" (id 1) (at 182.245 106.6801 0)
+      (effects (font (size 1.27 1.27)) (justify right))
+    )
+    (property "Footprint" "Connector_PinSocket_2.54mm:PinSocket_1x06_P2.54mm_Vertical" (id 2) (at 180.975 109.22 0)
+      (effects (font (size 1.27 1.27)) hide)
+    )
+    (property "Datasheet" "~" (id 3) (at 180.975 109.22 0)
+      (effects (font (size 1.27 1.27)) hide)
+    )
+    (pin "1")
+    (pin "2")
+    (pin "3")
+    (pin "4")
+    (pin "5")
+    (pin "6")
   )
   (symbol (lib_id "Regulator_Linear:L7805") (at 149.86 153.67 0) (unit 1)
@@
     (pin "2")
   )
-  (symbol (lib_id "Connector:Conn_01x03_Male") (at 149.86 132.08 90) (mirror x) (unit 1)
-    (in_bom yes) (on_board yes) (fields_autoplaced)
-    (property "Reference" "J1" (id 0) (at 149.86 127 90))
-    (property "Value" "Power" (id 1) (at 149.86 129.54 90))
-    (property "Footprint" "Connector_PinSocket_2.54mm:PinSocket_1x03_P2.54mm_Vertical" (id 2) (at 149.86 132.08 0)
-      (effects (font (size 1.27 1.27)) hide)
-    )
-    (property "Datasheet" "~" (id 3) (at 149.86 132.08 0)
+  (symbol (lib_id "Connector:Conn_01x03_Male") (at 149.86 128.27 90) (mirror x) (unit 1)
+    (in_bom yes) (on_board yes) (fields_autoplaced)
+    (property "Reference" "J1" (id 0) (at 149.86 123.19 90))
+    (property "Value" "Power" (id 1) (at 149.86 125.73 90))
+    (property "Footprint" "Connector_PinSocket_2.54mm:PinSocket_1x03_P2.54mm_Vertical" (id 2) (at 149.86 128.27 0)
+      (effects (font (size 1.27 1.27)) hide)
+    )
+    (property "Datasheet" "~" (id 3) (at 149.86 128.27 0)
       (effects (font (size 1.27 1.27)) hide)
     )
@@
     (pin "1")
     (pin "2")
+  )
+  (symbol (lib_id "Connector:Conn_01x03_Male") (at 149.86 132.715 90) (mirror x) (unit 1)
+    (in_bom yes) (on_board yes) (fields_autoplaced)
+    (property "Reference" "J4" (id 0) (at 149.86 127.635 90))
+    (property "Value" "Power" (id 1) (at 149.86 130.175 90))
+    (property "Footprint" "Connector_PinSocket_2.54mm:PinSocket_1x03_P2.54mm_Vertical" (id 2) (at 149.86 132.715 0)
+      (effects (font (size 1.27 1.27)) hide)
+    )
+    (property "Datasheet" "~" (id 3) (at 149.86 132.715 0)
+      (effects (font (size 1.27 1.27)) hide)
+    )
+    (pin "1")
+    (pin "2")
+    (pin "3")
   )
   (symbol (lib_id "Connector:USB_B_Micro") (at 199.39 127 0) (mirror y) (unit 1)
@@
       (reference "J3") (unit 1) (value "USB_B_Micro") (footprint "Connector_USB:USB_Micro-AB_Molex_47590-0001")
     )
+    (path "/c64623ea-1b89-43ec-92c6-a2d8ff19adad"
+      (reference "J4") (unit 1) (value "Power") (footprint "Connector_PinSocket_2.54mm:PinSocket_1x03_P2.54mm_Vertical")
+    )
+    (path "/04748a16-5476-4809-b159-9184ff58426c"
+      (reference "J5") (unit 1) (value "PinOut") (footprint "Connector_PinSocket_2.54mm:PinSocket_1x06_P2.54mm_Vertical")
+    )
     (path "/bfb5e7c3-ec60-41c0-a79b-ada084d506c2"
